Commit message: change stl path to .. in urdf file

File: hardware/urdf/urdf/dk2.SLDASM.urdf (robot description, URDF)
Before this commit: robot dk2.SLDASM, 10 links, 9 joints
Links:
- link base_link: geometry collision mesh filename=../meshes/base_link.STL; visual mesh filename=../meshes/base_link.STL
- link finger_l: geometry collision mesh filename=../meshes/finger_l.STL; visual mesh filename=../meshes/finger_l.STL
- link finger_r: geometry collision mesh filename=../meshes/finger_r.STL; visual mesh filename=../meshes/finger_r.STL
- link gripper: geometry collision mesh filename=../meshes/gripper.STL; visual mesh filename=../meshes/gripper.STL
- link link1: geometry collision mesh filename=../meshes/link1.STL; visual mesh filename=../meshes/link1.STL
- link link2: geometry collision mesh filename=../meshes/link2.STL; visual mesh filename=../meshes/link2.STL
- link link3: geometry collision mesh filename=../meshes/link3.STL; visual mesh filename=../meshes/link3.STL
- link link4: geometry collision mesh filename=../meshes/link4.STL; visual mesh filename=../meshes/link4.STL
- link link5: geometry collision mesh filename=../meshes/link5.STL; visual mesh filename=../meshes/link5.STL
- link link6: geometry collision mesh filename=../meshes/link6.STL; visual mesh filename=../meshes/link6.STL
